Commit message: Refactor

File: src/driveguard_description/urdf/diff_drive/actuator/caster.urdf.xacro (robot description, xacro)
@@ -1,5 +1,5 @@
 <?xml version="1.0"?>
 <robot xmlns:xacro="http://www.ros.org/wiki/xacro">
-   <xacro:include filename="$(find driveguard_description)/urdf/driveguard/common_inertia.xacro" />
+   <xacro:include filename="$(find driveguard_description)/urdf/diff_drive/common_inertia.xacro" />
     <xacro:macro name="caster_xacro" params="caster_name xyz">
         <link name="${caster_name}_caster_link">

File: src/driveguard_description/urdf/diff_drive/actuator/wheel.urdf.xacro (robot description, xacro)
@@ -1,5 +1,5 @@
 <?xml version="1.0"?>
 <robot xmlns:xacro="http://www.ros.org/wiki/xacro">
-   <xacro:include filename="$(find driveguard_description)/urdf/driveguard/common_inertia.xacro" />
+   <xacro:include filename="$(find driveguard_description)/urdf/diff_drive/common_inertia.xacro" />
     <xacro:macro name="wheel_xacro" params="wheel_name xyz">
         <link name="${wheel_name}_wheel_link">

File: src/driveguard_description/urdf/diff_drive/base.urdf.xacro (robot description, xacro)
@@ -1,5 +1,5 @@
 <?xml version="1.0"?>
 <robot xmlns:xacro="http://www.ros.org/wiki/xacro">
-   <xacro:include filename="$(find driveguard_description)/urdf/driveguard/common_inertia.xacro" />
+   <xacro:include filename="$(find driveguard_description)/urdf/diff_drive/common_inertia.xacro" />
     <xacro:macro name="base_xacro" params="length radius">
      <link name="base_footprint" />

File: src/driveguard_description/urdf/diff_drive/diff_drive.ros2_control.xacro (robot description, xacro)
@@ -1,5 +1,5 @@
 <?xml version="1.0"?>
 <robot xmlns:xacro="http://www.ros.org/wiki/xacro">
-    <xacro:macro name="driveguard_ros2_control">
+    <xacro:macro name="diff_drive_ros2_control">
     <ros2_control name="driveguardGazeboSystem" type="system">
             <hardware>
@@ -35,5 +35,5 @@
         <gazebo>
         <plugin filename="libgazebo_ros2_control.so" name="gazebo_ros2_control">
-            <parameters>$(find driveguard_description)/config/driveguard_ros2_controller.yaml</parameters>
+            <parameters>$(find driveguard_description)/config/diff_drive_ros2_controller.yaml</parameters>
             <ros>
                 <remapping>/driveguard_diff_drive_controller/cmd_vel_unstamped:=/cmd_vel</remapping>

File: src/driveguard_description/urdf/diff_drive/sensor/camera.urdf.xacro (robot description, xacro)
@@ -1,5 +1,5 @@
 <?xml version="1.0"?>
 <robot xmlns:xacro="http://www.ros.org/wiki/xacro">
-   <xacro:include filename="$(find driveguard_description)/urdf/driveguard/common_inertia.xacro" />
+   <xacro:include filename="$(find driveguard_description)/urdf/diff_drive/common_inertia.xacro" />
     <xacro:macro name="camera_xacro" params="xyz">
         <!-- ============相机模块================ -->

File: src/driveguard_description/urdf/diff_drive/sensor/imu.urdf.xacro (robot description, xacro)
@@ -1,5 +1,5 @@
 <?xml version="1.0"?>
 <robot xmlns:xacro="http://www.ros.org/wiki/xacro">
-   <xacro:include filename="$(find driveguard_description)/urdf/driveguard/common_inertia.xacro" />
+   <xacro:include filename="$(find driveguard_description)/urdf/diff_drive/common_inertia.xacro" />
     <xacro:macro name="imu_xacro" params="xyz">
         <link name="imu_link">

File: src/driveguard_description/urdf/diff_drive/sensor/laser.urdf.xacro (robot description, xacro)
@@ -1,5 +1,5 @@
 <?xml version="1.0"?>
 <robot xmlns:xacro="http://www.ros.org/wiki/xacro">
-   <xacro:include filename="$(find driveguard_description)/urdf/driveguard/common_inertia.xacro" />
+   <xacro:include filename="$(find driveguard_description)/urdf/diff_drive/common_inertia.xacro" />
     <xacro:macro name="laser_xacro" params="xyz">
         <gazebo reference="laser_cylinder_link">
