Commit message: 1. 新增一个ackermann模型"racecar" 2.新增robot_locazlization平滑里程计 3.新增ackermann模型的nav2配置 4.Update README.md 5.文件重命名

File: src/driveguard_description/urdf/ackermann/ackermann_gazebo_core.urdf.xacro (robot description, xacro)
@@ -1,44 +1,44 @@
 <?xml version="1.0"?>
 <robot xmlns:xacro="http://www.ros.org/wiki/xacro">
-    <!-- GAZEBO COLOUR -->
-    <!-- Gazebo is unable to use the same <material> tags that are already in the URDF (that RViz
+  <!-- GAZEBO COLOUR -->
+  <!-- Gazebo is unable to use the same <material> tags that are already in the URDF (that RViz
     uses). -->
-    <!-- Instead, we need to add gazebo tags for our links that refer to Gazebo materials -->
-    <gazebo reference="chassis_link">
-        <material>Gazebo/White</material>
-        <mu1>0.5</mu1>
-        <mu2>0.5</mu2>
-    </gazebo>
-    <gazebo reference="fr_left_wheel_link">
-        <material>Gazebo/Grey</material>
-        <mu1>150.0</mu1>
-        <mu2>10.0</mu2>
-    </gazebo>
-    <gazebo reference="fr_right_wheel_link">
-        <material>Gazebo/Grey</material>
-        <mu1>150.0</mu1>
-        <mu2>10.0</mu2>
-    </gazebo>
-    <gazebo reference="re_left_wheel_link">
-        <material>Gazebo/Grey</material>
-        <mu1>150.0</mu1>
-        <mu2>10.0</mu2>
-    </gazebo>
-    <gazebo reference="re_right_wheel_link">
-        <material>Gazebo/Grey</material>
-        <mu1>150.0</mu1>
-        <mu2>10.0</mu2>
-    </gazebo>
-    <gazebo reference="virtual_steer_link">
-        <material>Gazebo/Yellow</material>
-    </gazebo>
-    <!-- LASER -->
-    <gazebo reference="laser_link">
-        <material>Gazebo/Black</material>
-        <mu1>1.0</mu1>
-        <mu2>1.0</mu2>
-    </gazebo>
-    <gazebo reference="laser_link">
-      <sensor name="laser_sensor" type="ray">
+  <!-- Instead, we need to add gazebo tags for our links that refer to Gazebo materials -->
+  <gazebo reference="chassis_link">
+    <material>Gazebo/White</material>
+    <mu1>0.5</mu1>
+    <mu2>0.5</mu2>
+  </gazebo>
+  <gazebo reference="fr_left_wheel_link">
+    <material>Gazebo/Grey</material>
+    <mu1>150.0</mu1>
+    <mu2>10.0</mu2>
+  </gazebo>
+  <gazebo reference="fr_right_wheel_link">
+    <material>Gazebo/Grey</material>
+    <mu1>150.0</mu1>
+    <mu2>10.0</mu2>
+  </gazebo>
+  <gazebo reference="re_left_wheel_link">
+    <material>Gazebo/Grey</material>
+    <mu1>150.0</mu1>
+    <mu2>10.0</mu2>
+  </gazebo>
+  <gazebo reference="re_right_wheel_link">
+    <material>Gazebo/Grey</material>
+    <mu1>150.0</mu1>
+    <mu2>10.0</mu2>
+  </gazebo>
+  <gazebo reference="virtual_steer_link">
+    <material>Gazebo/Yellow</material>
+  </gazebo>
+  <!-- LASER -->
+  <gazebo reference="laser_link">
+    <material>Gazebo/Black</material>
+    <mu1>1.0</mu1>
+    <mu2>1.0</mu2>
+  </gazebo>
+  <gazebo reference="laser_link">
+    <sensor name="laser_sensor" type="ray">
       <always_on>true</always_on>
       <visualize>false</visualize>
@@ -46,22 +46,22 @@
       <pose>0 0 0.2 0 0 0</pose>
       <ray>
-          <scan>
-            <horizontal>
-              <samples>360</samples>
-              <resolution>1.000000</resolution>
-              <min_angle>0.000000</min_angle>
-              <max_angle>6.280000</max_angle>
-            </horizontal>
-          </scan>
-          <range>
-            <min>0.5000</min>
-            <max>10.5</max>
-            <resolution>0.015000</resolution>
-          </range>
-          <noise>
-            <type>gaussian</type>
-            <mean>0.0</mean>
-            <stddev>0.01</stddev>
-          </noise>
+        <scan>
+          <horizontal>
+            <samples>360</samples>
+            <resolution>1.000000</resolution>
+            <min_angle>0.000000</min_angle>
+            <max_angle>6.280000</max_angle>
+          </horizontal>
+        </scan>
+        <range>
+          <min>0.5000</min>
+          <max>10.5</max>
+          <resolution>0.015000</resolution>
+        </range>
+        <noise>
+          <type>gaussian</type>
+          <mean>0.0</mean>
+          <stddev>0.01</stddev>
+        </noise>
       </ray>
       <plugin name="laserscan" filename="libgazebo_ros_ray_sensor.so">
@@ -72,177 +72,177 @@
         <frame_name>laser_link</frame_name>
       </plugin>
-      </sensor>
-    </gazebo>
-    <gazebo reference="imu_link">
-        <material>Gazebo/Black</material>
-        <mu1>1.0</mu1>
-        <mu2>1.0</mu2>
-    </gazebo>
-    <gazebo reference="imu_link">
-      <sensor name="imu_sensor" type="imu">
+    </sensor>
+  </gazebo>
+  <gazebo reference="imu_link">
+    <material>Gazebo/Black</material>
+    <mu1>1.0</mu1>
+    <mu2>1.0</mu2>
+  </gazebo>
+  <gazebo reference="imu_link">
+    <sensor name="imu_sensor" type="imu">
       <plugin filename="libgazebo_ros_imu_sensor.so" name="imu_plugin">
-          <ros>
-            <namespace>/</namespace>
-            <remapping>~/out:=imu</remapping>
-          </ros>
-          <initial_orientation_as_reference>false</initial_orientation_as_reference>
-        </plugin>
-        <always_on>true</always_on>
-        <update_rate>100</update_rate>
-        <visualize>true</visualize>
-        <imu>
-          <angular_velocity>
-            <x>
-              <noise type="gaussian">
-                <mean>0.0</mean>
-                <stddev>2e-4</stddev>
-                <bias_mean>0.0000075</bias_mean>
-                <bias_stddev>0.0000008</bias_stddev>
-              </noise>
-            </x>
-            <y>
-              <noise type="gaussian">
-                <mean>0.0</mean>
-                <stddev>2e-4</stddev>
-                <bias_mean>0.0000075</bias_mean>
-                <bias_stddev>0.0000008</bias_stddev>
-              </noise>
-            </y>
-            <z>
-              <noise type="gaussian">
-                <mean>0.0</mean>
-                <stddev>2e-4</stddev>
-                <bias_mean>0.0000075</bias_mean>
-                <bias_stddev>0.0000008</bias_stddev>
-              </noise>
-            </z>
-          </angular_velocity>
-          <linear_acceleration>
-            <x>
-              <noise type="gaussian">
-                <mean>0.0</mean>
-                <stddev>1.7e-2</stddev>
-                <bias_mean>0.1</bias_mean>
-                <bias_stddev>0.001</bias_stddev>
-              </noise>
-            </x>
-            <y>
-              <noise type="gaussian">
-                <mean>0.0</mean>
-                <stddev>1.7e-2</stddev>
-                <bias_mean>0.1</bias_mean>
-                <bias_stddev>0.001</bias_stddev>
-              </noise>
-            </y>
-            <z>
-              <noise type="gaussian">
-                <mean>0.0</mean>
-                <stddev>1.7e-2</stddev>
-                <bias_mean>0.1</bias_mean>
-                <bias_stddev>0.001</bias_stddev>
-              </noise>
-            </z>
-          </linear_acceleration>
-        </imu>
-      </sensor>
-    </gazebo>
-    <!-- JOINT STATE PUBLISHER -->
-    <!-- Gazebo requires the use of plugins to interact with other systems such as ROS. -->
-    <!-- This plugin will publish the joint_states for the selected joints
+        <ros>
+          <namespace>/</namespace>
+          <remapping>~/out:=imu</remapping>
+        </ros>
+        <initial_orientation_as_reference>false</initial_orientation_as_reference>
+      </plugin>
+      <always_on>true</always_on>
+      <update_rate>100</update_rate>
+      <visualize>true</visualize>
+      <imu>
+        <angular_velocity>
+          <x>
+            <noise type="gaussian">
+              <mean>0.0</mean>
+              <stddev>2e-4</stddev>
+              <bias_mean>0.0000075</bias_mean>
+              <bias_stddev>0.0000008</bias_stddev>
+            </noise>
+          </x>
+          <y>
+            <noise type="gaussian">
+              <mean>0.0</mean>
+              <stddev>2e-4</stddev>
+              <bias_mean>0.0000075</bias_mean>
+              <bias_stddev>0.0000008</bias_stddev>
+            </noise>
+          </y>
+          <z>
+            <noise type="gaussian">
+              <mean>0.0</mean>
+              <stddev>2e-4</stddev>
+              <bias_mean>0.0000075</bias_mean>
+              <bias_stddev>0.0000008</bias_stddev>
+            </noise>
+          </z>
+        </angular_velocity>
+        <linear_acceleration>
+          <x>
+            <noise type="gaussian">
+              <mean>0.0</mean>
+              <stddev>1.7e-2</stddev>
+              <bias_mean>0.1</bias_mean>
+              <bias_stddev>0.001</bias_stddev>
+            </noise>
+          </x>
+          <y>
+            <noise type="gaussian">
+              <mean>0.0</mean>
+              <stddev>1.7e-2</stddev>
+              <bias_mean>0.1</bias_mean>
+              <bias_stddev>0.001</bias_stddev>
+            </noise>
+          </y>
+          <z>
+            <noise type="gaussian">
+              <mean>0.0</mean>
+              <stddev>1.7e-2</stddev>
+              <bias_mean>0.1</bias_mean>
+              <bias_stddev>0.001</bias_stddev>
+            </noise>
+          </z>
+        </linear_acceleration>
+      </imu>
+    </sensor>
+  </gazebo>
+  <!-- JOINT STATE PUBLISHER -->
+  <!-- Gazebo requires the use of plugins to interact with other systems such as ROS. -->
+  <!-- This plugin will publish the joint_states for the selected joints
             (which robot_state_publisher can then use to broadcast the approprate tf).
          Using Gazebo ROS2 control plugin (ros2_control) (part of ROS2 control system) publishing and
     control of joint.-->
-    <gazebo>
-        <plugin name="gazebo_ros_joint_state_publisher"
-            filename="libgazebo_ros_joint_state_publisher.so">
-            <update_rate>100</update_rate>
-            <joint_name>fr_right_steer_joint</joint_name>
-            <joint_name>fr_right_wheel_joint</joint_name>
-            <joint_name>fr_left_steer_joint</joint_name>
-            <joint_name>fr_left_wheel_joint</joint_name>
-            <joint_name>re_right_wheel_joint</joint_name>
-            <joint_name>re_left_wheel_joint</joint_name>
-            <joint_name>virtual_steering_wheel_joint</joint_name>
-        </plugin>
-    </gazebo>
-    <!-- This plugin will read a JointTrajectory message from the /set_joint_trajectory topic
+  <gazebo>
+    <plugin name="gazebo_ros_joint_state_publisher"
+      filename="libgazebo_ros_joint_state_publisher.so">
+      <update_rate>100</update_rate>
+      <joint_name>fr_right_steer_joint</joint_name>
+      <joint_name>fr_right_wheel_joint</joint_name>
+      <joint_name>fr_left_steer_joint</joint_name>
+      <joint_name>fr_left_wheel_joint</joint_name>
+      <joint_name>re_right_wheel_joint</joint_name>
+      <joint_name>re_left_wheel_joint</joint_name>
+      <joint_name>virtual_steering_wheel_joint</joint_name>
+    </plugin>
+  </gazebo>
+  <!-- This plugin will read a JointTrajectory message from the /set_joint_trajectory topic
             and move the machine accordingly. It's a bit clunky but it works. -->
-    <!-- You'll probably want to add damping to the joints to stop them it flopping around.
+  <!-- You'll probably want to add damping to the joints to stop them it flopping around.
             e.g. <dynamics damping="10.0" friction="10.0"/> -->
-    <!-- Here's an example message to publish to test it:
+  <!-- Here's an example message to publish to test it:
             ros2 topic pub -1 /set_joint_trajectory trajectory_msgs/msg/JointTrajectory  '{header: {frame_id:
     world}, joint_names: [slider_joint, arm_joint], points: [  {positions: {0.8,0.6}} ]}' -->
-    <gazebo>
-        <plugin name="gazebo_ros_joint_pose_trajectory"
-            filename="libgazebo_ros_joint_pose_trajectory.so">
-            <update_rate>2</update_rate>
-        </plugin>
-    </gazebo>
-    <!-- ACKERMANN DRIVE PLUGIN -->
-    <gazebo>
-        <plugin name='gazebo_ackermann_drive' filename='libgazebo_ros_ackermann_drive.so'>
-            <ros>
-                <!-- <namespace>ugv_gazebo_ackermann</namespace> -->
-                <remapping>cmd_vel:=cmd_vel</remapping>
-                <remapping>odom:=odom</remapping>
-                <remapping>distance:=distance</remapping>
-            </ros>
-            <update_rate>100.0</update_rate>
-            <!-- wheels -->
-            <front_left_joint>fr_left_wheel_joint</front_left_joint>
-            <front_right_joint>fr_right_wheel_joint</front_right_joint>
-            <rear_left_joint>re_left_wheel_joint</rear_left_joint>
-            <rear_right_joint>re_right_wheel_joint</rear_right_joint>
-            <left_steering_joint>fr_left_steer_joint</left_steering_joint>
-            <right_steering_joint>fr_right_steer_joint</right_steering_joint>
-            <steering_wheel_joint>virtual_steering_wheel_joint</steering_wheel_joint>
-            <!-- Max absolute steer angle for tyre in radians-->
-            <!-- Any cmd_vel angular z greater than this would be capped -->
-            <max_steer>0.383972</max_steer>
-            <!-- Max absolute steering angle of steering wheel -->
-            <max_steering_angle>1.570796</max_steering_angle>
-            <!-- Max absolute linear speed in m/s -->
-            <max_speed>5</max_speed>
-            <!-- PID tuning -->
-            <left_steering_pid_gain>1500 0 1</left_steering_pid_gain>
-            <left_steering_i_range>0 0</left_steering_i_range>
-            <right_steering_pid_gain>1500 0 1</right_steering_pid_gain>
-            <right_steering_i_range>0 0</right_steering_i_range>
-            <linear_velocity_pid_gain>1500 0 1</linear_velocity_pid_gain>
-            <linear_velocity_i_range>0 0</linear_velocity_i_range>
-            <!-- output -->
-            <publish_odom>true</publish_odom>
-            <publish_odom_tf>true</publish_odom_tf>     <!-- Don't pubslish this when using robot
+  <gazebo>
+    <plugin name="gazebo_ros_joint_pose_trajectory"
+      filename="libgazebo_ros_joint_pose_trajectory.so">
+      <update_rate>2</update_rate>
+    </plugin>
+  </gazebo>
+  <!-- ACKERMANN DRIVE PLUGIN -->
+  <gazebo>
+    <plugin name='gazebo_ackermann_drive' filename='libgazebo_ros_ackermann_drive.so'>
+      <ros>
+        <!-- <namespace>ugv_gazebo_ackermann</namespace> -->
+        <remapping>cmd_vel:=cmd_vel</remapping>
+        <remapping>odom:=odom</remapping>
+        <remapping>distance:=distance</remapping>
+      </ros>
+      <update_rate>100.0</update_rate>
+      <!-- wheels -->
+      <front_left_joint>fr_left_wheel_joint</front_left_joint>
+      <front_right_joint>fr_right_wheel_joint</front_right_joint>
+      <rear_left_joint>re_left_wheel_joint</rear_left_joint>
+      <rear_right_joint>re_right_wheel_joint</rear_right_joint>
+      <left_steering_joint>fr_left_steer_joint</left_steering_joint>
+      <right_steering_joint>fr_right_steer_joint</right_steering_joint>
+      <steering_wheel_joint>virtual_steering_wheel_joint</steering_wheel_joint>
+      <!-- Max absolute steer angle for tyre in radians-->
+      <!-- Any cmd_vel angular z greater than this would be capped -->
+      <max_steer>0.383972</max_steer>
+      <!-- Max absolute steering angle of steering wheel -->
+      <max_steering_angle>1.570796</max_steering_angle>
+      <!-- Max absolute linear speed in m/s -->
+      <max_speed>5</max_speed>
+      <!-- PID tuning -->
+      <left_steering_pid_gain>1500 0 1</left_steering_pid_gain>
+      <left_steering_i_range>0 0</left_steering_i_range>
+      <right_steering_pid_gain>1500 0 1</right_steering_pid_gain>
+      <right_steering_i_range>0 0</right_steering_i_range>
+      <linear_velocity_pid_gain>1500 0 1</linear_velocity_pid_gain>
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